File: hardware/kicad/Pico1541/_autosave-Pico1541.kicad_pcb (KiCad board)
At the start: 2 copper layers, 100 x 76.2 mm, 62 parts, among them J1 SWD, J2 Serial, J3 Display/Keys, J4 Micro SD Card, J5 5V_EXT, J6 USB_A, J7 OLED/Key_Hat, J8 OLED, J9 DIN-6, Q1 MMBT3904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

Commit message: feat(pio): output SYNC state to GPIO 10 directly from PIO
Connections:
- U2 pad 5: +5V -> unconnected-(U2-VP-Pad5)
Routing:
- net Net-(D3-KA): track 0.00 -> 15.3 mm
- net /PLED_N: track 65.1 -> 79.2 mm
- net Net-(D2-GA): track 0.00 -> 9.75 mm
- net Net-(D2-RA): track 0.00 -> 8.71 mm
- net Net-(D2-BA): track 0.00 -> 8.53 mm
- net +5V: track 166.2 -> 160.5 mm, vias 3 -> 2
- net GND: vias 389 -> 394
Changed lines of the file:
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@@
 			(layers "F.Cu" "F.Mask" "F.Paste")
 			(roundrect_rratio 0.25)
-			(net "+5V")
+			(net "unconnected-(U2-VP-Pad5)")
 			(pinfunction "VP_5")
-			(pintype "passive")
+			(pintype "passive+no_connect")
 		)
 		(pad "6" smd roundrect
@@
 	)
 	(via
+		(at 112.6 119.95)
+		(size 0.8)
+		(drill 0.4)
+		(layers "F.Cu" "B.Cu")
+		(free yes)
+		(net "GND")
+	)
+	(via
 		(at 109.73 68.53)
 		(size 0.8)
@@
 	)
 	(via
+		(at 114.6 120.05)
+		(size 0.8)
+		(drill 0.4)
+		(layers "F.Cu" "B.Cu")
+		(free yes)
+		(net "GND")
+	)
+	(via
 		(at 138.9 114.85)
 		(size 0.8)
@@
 	)
 	(via
+		(at 112.6 122.15)
+		(size 0.8)
+		(drill 0.4)
+		(layers "F.Cu" "B.Cu")
+		(free yes)
+		(net "GND")
+	)
+	(via
 		(at 148.8 106.55)
 		(size 0.8)
@@
 	)
 	(via
+		(at 110.8 122.1)
+		(size 0.8)
+		(drill 0.4)
+		(layers "F.Cu" "B.Cu")
+		(free yes)
+		(net "GND")
+	)
+	(via
 		(at 159.1 104.95)
 		(size 0.8)
@@
 	)
 	(via
-		(at 116.6 117.75)
-		(size 0.8)
-		(drill 0.4)
-		(layers "F.Cu" "B.Cu")
-		(free yes)
-		(net "GND")
-	)
-	(via
 		(at 104.3 78.81)
 		(size 0.8)
@@
 	)
 	(via
+		(at 114.85 127.3)
+		(size 0.8)
+		(drill 0.4)
+		(layers "F.Cu" "B.Cu")
+		(free yes)
+		(net "GND")
+	)
+	(via
+		(at 114.6 123.55)
+		(size 0.8)
+		(drill 0.4)
+		(layers "F.Cu" "B.Cu")
+		(free yes)
+		(net "GND")
+	)
+	(via
 		(at 141 70.15)
 		(size 0.8)
@@
 	)
 	(segment
-		(start 153 75.1)
-		(end 154.3625 75.1)
-		(width 0.5)
-		(layer "F.Cu")
-		(net "+5V")
-	)
-	(segment
 		(start 156.45 89.88)
 		(end 156.45 89.1625)
@@
 	)
 	(via
-		(at 153 75.1)
-		(size 0.8)
-		(drill 0.4)
-		(layers "F.Cu" "B.Cu")
-		(net "+5V")
-	)
-	(via
 		(at 119.25849 64.255283)
 		(size 0.8)
@@
 	)
 	(segment
-		(start 150.35 75.1)
-		(end 153 75.1)
-		(width 0.5)
-		(layer "B.Cu")
-		(net "+5V")
-	)
-	(segment
-		(start 150.35 75.1)
-		(end 149.75 75.1)
-		(width 0.5)
-		(layer "B.Cu")
-		(net "+5V")
-	)
-	(segment
 		(start 147.617874 72.967874)
 		(end 147.617874 63.132126)
@@
 	)
 	(segment
-		(start 149.4 78.65)
-		(end 149.4 75.2)
-		(width 0.5)
-		(layer "B.Cu")
-		(net "+5V")
-	)
-	(segment
-		(start 149.5 75.1)
-		(end 150.35 75.1)
+		(start 147.617874 63.132126)
+		(end 148.4 62.35)
 		(width 0.5)
 		(layer "B.Cu")
@@
 	)
 	(segment
-		(start 147.617874 63.132126)
-		(end 148.4 62.35)
+		(start 149.4 78.65)
+		(end 149.4 74.75)
 		(width 0.5)
 		(layer "B.Cu")
@@
 	)
 	(segment
-		(start 149.75 75.1)
-		(end 147.617874 72.967874)
-		(width 0.5)
-		(layer "B.Cu")
-		(net "+5V")
-	)
-	(segment
 		(start 148.65 60.65)
 		(end 148.4 60.65)
@@
 	)
 	(segment
-		(start 127.202082 58.25)
-		(end 121.352082 64.1)
+		(start 149.4 74.75)
+		(end 147.617874 72.967874)
 		(width 0.5)
 		(layer "B.Cu")
@@
 	)
 	(segment
-		(start 149.4 75.2)
-		(end 149.5 75.1)
+		(start 127.202082 58.25)
+		(end 121.352082 64.1)
 		(width 0.5)
 		(layer "B.Cu")
@@
 	)
 	(segment
-		(start 127.125 83.925)
-		(end 128.55 82.5)
+		(start 120.275 125.325)
+		(end 120.275 124.9)
 		(width 0.25)
 		(layer "F.Cu")
-		(net "/PLED_N")
+		(net "Net-(D3-KA)")
 	)
 	(segment
-		(start 125.991666 83.92)
-		(end 125.996666 83.925)
+		(start 114.4 118.1)
+		(end 115.55 119.25)
 		(width 0.25)
 		(layer "F.Cu")
-		(net "/PLED_N")
+		(net "Net-(D3-KA)")
 	)
 	(segment
-		(start 107.944292 114.305708)
-		(end 118.7 103.55)
+		(start 115.55 119.25)
+		(end 115.55 125.65)
+		(width 0.25)
+		(layer "F.Cu")
+		(net "Net-(D3-KA)")
+	)
+	(segment
+		(start 115.55 125.65)
+		(end 116.9 127)
+		(width 0.25)
+		(layer "F.Cu")
+		(net "Net-(D3-KA)")
+	)
+	(segment
+		(start 118.6 127)
+		(end 120.275 125.325)
+		(width 0.25)
+		(layer "F.Cu")
+		(net "Net-(D3-KA)")
+	)
+	(segment
+		(start 116.9 127)
+		(end 118.6 127)
+		(width 0.25)
+		(layer "F.Cu")
+		(net "Net-(D3-KA)")
+	)
+	(segment
+		(start 114.4 117.25)
+		(end 114.4 118.1)
+		(width 0.25)
+		(layer "F.Cu")
+		(net "Net-(D3-KA)")
+	)
+	(segment
+		(start 117.75 119.25)
+		(end 117.735 119.265)
 		(width 0.25)
 		(layer "F.Cu")
@@
 	)
 	(segment
-		(start 122.979804 83.92)
-		(end 125.991666 83.92)
+		(start 115.35 116.35)
+		(end 117.75 118.75)
 		(width 0.25)
 		(layer "F.Cu")
@@
 	)
 	(segment
-		(start 118.7 103.55)
-		(end 118.7 85.859188)
+		(start 111.35 116.35)
+		(end 115.35 116.35)
 		(width 0.25)
 		(layer "F.Cu")
@@
 	)
 	(segment
-		(start 126.93 64.88)
-		(end 124.31 64.88)
+		(start 125.991666 83.92)
+		(end 125.996666 83.925)
+		(width 0.25)
+		(layer "F.Cu")
+		(net "/PLED_N")
+	)
+	(segment
+		(start 117.735 119.265)
+		(end 117.735 124.9)
 		(width 0.25)
 		(layer "F.Cu")
@@
 	)
 	(segment
-		(start 120.634188 83.925)
-		(end 122.974804 83.925)
+		(start 127.125 83.925)
+		(end 128.55 82.5)
 		(width 0.25)
 		(layer "F.Cu")
@@
 	)
 	(segment
+		(start 117.75 118.75)
+		(end 117.75 119.25)
+		(width 0.25)
+		(layer "F.Cu")
+		(net "/PLED_N")
+	)
+	(segment
+		(start 122.979804 83.92)
+		(end 125.991666 83.92)
+		(width 0.25)
+		(layer "F.Cu")
+		(net "/PLED_N")
+	)
+	(segment
+		(start 126.93 64.88)
+		(end 124.31 64.88)
+		(width 0.25)
+		(layer "F.Cu")
+		(net "/PLED_N")
+	)
+	(segment
+		(start 120.634188 83.925)
+		(end 122.974804 83.925)
+		(width 0.25)
+		(layer "F.Cu")
+		(net "/PLED_N")
+	)
+	(segment
 		(start 118.7 85.859188)
 		(end 120.634188 83.925)
@@
 	)
 	(segment
+		(start 111.35 116.35)
+		(end 111.35 110.9)
+		(width 0.25)
+		(layer "F.Cu")
+		(net "/PLED_N")
+	)
+	(segment
+		(start 118.7 103.55)
+		(end 118.7 85.859188)
+		(width 0.25)
+		(layer "F.Cu")
+		(net "/PLED_N")
+	)
+	(segment
+		(start 111.35 110.9)
+		(end 118.7 103.55)
+		(width 0.25)
+		(layer "F.Cu")
+		(net "/PLED_N")
+	)
+	(segment
 		(start 124.31 54.72)
 		(end 124.305 54.725)
@@
 	)
 	(segment
+		(start 109.15 121.2)
+		(end 108.076 122.274)
+		(width 0.25)
+		(layer "F.Cu")
+		(net "Net-(D2-BA)")
+	)
+	(segment
+		(start 109.15 121.163604)
+		(end 109.15 121.2)
+		(width 0.25)
+		(layer "F.Cu")
+		(net "Net-(D2-BA)")
+	)
+	(segment
+		(start 108.076 122.274)
+		(end 108.076 124.15)
+		(width 0.25)
+		(layer "F.Cu")
+		(net "Net-(D2-BA)")
+	)
+	(segment
+		(start 112 118.313604)
+		(end 109.15 121.163604)
+		(width 0.25)
+		(layer "F.Cu")
+		(net "Net-(D2-BA)")
+	)
+	(segment
+		(start 112 117.25)
+		(end 112 118.313604)
+		(width 0.25)
+		(layer "F.Cu")
+		(net "Net-(D2-BA)")
+	)
+	(segment
+		(start 109.6 125.674)
+		(end 109.6 121.35)
+		(width 0.25)
+		(layer "F.Cu")
+		(net "Net-(D2-GA)")
+	)
+	(segment
+		(start 109.6 121.35)
+		(end 112.8 118.15)
+		(width 0.25)
+		(layer "F.Cu")
+		(net "Net-(D2-GA)")
+	)
+	(segment
+		(start 112.8 118.15)
+		(end 112.8 117.25)
+		(width 0.25)
+		(layer "F.Cu")
+		(net "Net-(D2-GA)")
+	)
+	(segment
+		(start 113.6 124.976)
+		(end 112.902 125.674)
+		(width 0.25)
+		(layer "F.Cu")
+		(net "Net-(D2-RA)")
+	)
+	(segment
+		(start 113.6 117.25)
+		(end 113.6 124.976)
+		(width 0.25)
+		(layer "F.Cu")
+		(net "Net-(D2-RA)")
+	)
+	(segment
